File: Smart Buck Converter/Buck Conversion.kicad_sch (KiCad schematic)
At the start: 25 parts, among them Q1 IRFR9220TRPBF-BE3, U1 LM2596S-ADJ, U3 AP2204K-3.3, U6 STCS05DR

Commit message: Revision 2 update
Regenerated gerber files to rev 2 design, made minor changes to PCB layout before exporting. Changed I2C interface connector from 4-pin right angle style to vertical style, added the new connector the the KiCad footprints library.
Parts:
- D1: value PMEG3015EH -> CDBMHT340-HF
Changed lines of the file:
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@@
+    )
+  )
+  (symbol (lib_id "Diode:PMEG3015EH") (at 187.96 34.29 180) (unit 1)
+    (in_bom yes) (on_board yes) (dnp no)
+    (property "Reference" "D1" (at 187.96 29.21 0)
+      (effects (font (size 1.27 1.27)))
+    )
+    (property "Value" "CDBMHT340-HF" (at 187.96 31.75 0)
+      (effects (font (size 1.27 1.27)))
+    )
+    (property "Footprint" "Diode_SMD:D_SOD-123F" (at 187.96 29.845 0)
+      (effects (font (size 1.27 1.27)) hide)
+    )
+    (property "Datasheet" "https://www.mouser.com/datasheet/2/80/comchip_technology_comc-s-a0004994317-1-1734023.pdf" (at 187.96 34.29 0)
+      (effects (font (size 1.27 1.27)) hide)
+    )
+    (pin "1")
+    (pin "2")
+    (instances
+      (project "Smart Buck Converter"
+        (path "/e63e39d7-6ac0-4ffd-8aa3-1841a4541b55/039da05a-c514-47d5-a2ac-898f12b81897"
+          (reference "D1") (unit 1)
+        )
+        (path "/e63e39d7-6ac0-4ffd-8aa3-1841a4541b55/f42437d8-c8e9-4867-9848-3b4f9584cf8b"
+          (reference "D6") (unit 1)
+        )
+      )
     )
   )
@@
         )
       )
-    )
-  )
-  (symbol (lib_id "Diode:PMEG3015EH") (at 187.96 34.29 180) (unit 1)
-    (in_bom yes) (on_board yes) (dnp no)
-    (property "Reference" "D1" (at 187.96 29.21 0)
-      (effects (font (size 1.27 1.27)))
-    )
-    (property "Value" "PMEG3015EH" (at 187.96 31.75 0)
-      (effects (font (size 1.27 1.27)))
-    )
-    (property "Footprint" "Diode_SMD:D_SOD-123F" (at 187.96 29.845 0)
-      (effects (font (size 1.27 1.27)) hide)
-    )
-    (property "Datasheet" "https://assets.nexperia.com/documents/data-sheet/PMEG3015EH_EJ.pdf" (at 187.96 34.29 0)
-      (effects (font (size 1.27 1.27)) hide)
-    )
-    (pin "1")
-    (pin "2")
-    (instances
-      (project "Smart Buck Converter"
-        (path "/e63e39d7-6ac0-4ffd-8aa3-1841a4541b55/039da05a-c514-47d5-a2ac-898f12b81897"
-          (reference "D1") (unit 1)
-        )
-        (path "/e63e39d7-6ac0-4ffd-8aa3-1841a4541b55/f42437d8-c8e9-4867-9848-3b4f9584cf8b"
-          (reference "D6") (unit 1)
-        )
-      )
